File: Expansion_Bay_FW16_Oculink8.kicad_sch (KiCad schematic)
At the start: 6 parts, among them J1 FAN1, J2 OCuLink_8i, J3 FW_EBI, J5 FAN0

Commit message: Add files via upload
Connections:
- net at J3.SB6 (PEX_RX3P): now also J2.A17 (PEX_RX3P)
- net at J3.SL6 (PEX_TX3P): now also J2.B17 (PEX_TX3P)
Changed lines of the file:
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@@
-	(wire
-		(pts
-			(xy 246.38 317.5) (xy 344.17 317.5)
-		)
-		(stroke
-			(width 0)
-			(type default)
-		)
-	)
 	(wire
 		(pts
@@
 	(wire
 		(pts
-			(xy 383.54 318.77) (xy 383.54 302.26)
-		)
-		(stroke
-			(width 0)
-			(type default)
-		)
-	)
-	(wire
-		(pts
 			(xy 331.47 275.59) (xy 331.47 270.51)
 		)
@@
 	(wire
 		(pts
+			(xy 246.38 200.66) (xy 246.38 318.77)
+		)
+		(stroke
+			(width 0)
+			(type default)
+		)
+	)
+	(wire
+		(pts
 			(xy 259.08 200.66) (xy 259.08 334.01)
 		)
@@
 	(wire
 		(pts
+			(xy 289.56 200.66) (xy 289.56 219.71)
+		)
+		(stroke
+			(width 0)
+			(type default)
+		)
+	)
+	(wire
+		(pts
 			(xy 353.06 179.07) (xy 350.52 179.07)
 		)
@@
 	(wire
 		(pts
+			(xy 246.38 318.77) (xy 336.55 318.77)
+		)
+		(stroke
+			(width 0)
+			(type default)
+		)
+	)
+	(wire
+		(pts
 			(xy 303.53 303.53) (xy 303.53 307.34)
 		)
@@
 	(wire
 		(pts
-			(xy 246.38 200.66) (xy 246.38 317.5)
-		)
-		(stroke
-			(width 0)
-			(type default)
-		)
-	)
-	(wire
-		(pts
 			(xy 334.01 303.53) (xy 334.01 307.34)
 		)
@@
 	(wire
 		(pts
-			(xy 289.56 201.93) (xy 289.56 219.71)
-		)
-		(stroke
-			(width 0)
-			(type default)
-		)
-	)
-	(wire
-		(pts
 			(xy 372.11 303.53) (xy 372.11 307.34)
 		)
@@
 		)
 		(stroke
+			(width 0)
+			(type default)
+		)
+	)
+	(wire
+		(pts
+			(xy 336.55 303.53) (xy 336.55 318.77)
+		)
+		(stroke
